File: electronique/schematic_draft/tom&Jerry_Draft/STM32x.kicad_sch (KiCad schematic)
At the start: 27 parts, among them J1 Conn_02x07_Odd_Even, SW1 SW_Push, SW2 SW_Push, SW3 SW_Push, SW4 SW_Push, Y1 16MHz

Commit message: STM32 KiCAD V1
Parts:
- added IC4: STM32G431CBU3, QFN50P700X700X65-49N-D, symbol STM32G431CBU3:STM32G431CBU3
- added R22: 100k, symbol Device:R
Connections:
- net +3.3V: now also IC4.1 (VBAT), IC4.20 (VREF+), IC4.21 (VDDA), IC4.23 (VDD_1), IC4.35 (VDD_2), IC4.48 (VDD_3)
- net GND: now also IC4.49 (VSS), R22.1
- net NRST: now also IC4.7 (PG10-NRST)
- net OSC_IN: now also IC4.5 (PF0-OSC_IN)
- net OSC_OUT: now also IC4.6 (PF1-OSC_OUT)
- net STLINK_SWO: now reaches J1.8 (Pin_8)
- net STLINK_SWO: now also IC4.41 (PB3)
- net RX renamed VCP_RX
- net VCP_RX: now also IC4.31 (PA9)
- net SWCLK renamed STLINK_SWCLK
- net STLINK_SWCLK: now also IC4.37 (PA14)
- net SWDIO renamed STLINK_SWDIO
- net STLINK_SWDIO: now also IC4.36 (PA13)
- net TX renamed VCP_TX
- net VCP_TX: now also IC4.32 (PA10)
- new net: IC4.46 (PB8-BOOT0), R22.2
- new net DRIVER_1_FWD: IC4.17 (PB0)
- new net DRIVER_1_REV: IC4.18 (PB1)
- new net DRIVER_2_FWD: IC4.22 (PB10)
- new net DRIVER_2_REV: IC4.24 (PB11)
- new net IMU_INT1: IC4.16 (PC4)
- new net IMU_INT2: IC4.19 (PB2)
- new net IMU_MISO/SDO: IC4.14 (PA6)
- new net IMU_MOSI/SDIO: IC4.15 (PA7)
- new net IMU_SCLK: IC4.13 (PA5)
- new net LIDAR_M_CTR: IC4.8 (PA0)
- new net LIDAR_RX: IC4.11 (PA3)
- new net LIDAR_TX: IC4.10 (PA2)
- new net ODOM2_PHASEA: IC4.39 (PC10)
- new net ODOM2_PHASEB: IC4.38 (PA15)
- new net ODOM_PHASEA: IC4.45 (PB7)
- new net ODOM_PHASEB: IC4.44 (PB6)
- new net TOF_GPIO1: IC4.43 (PB5)
- new net TOF_SCL: IC4.30 (PA8)
- new net TOF_SDA: IC4.40 (PC11)
- new net TOF_XSHUT: IC4.42 (PB4)
- no-connect marks 5 -> 17
Other:
- note added: "AJouter des patines de test en sortie de tout les I/O du STM32"
- note added: "mauvaise ref de composant voir STDC14"

Commit message: STM32 KiCAD V2 - 18.09.2024
Parts:
- removed D1: LED_ON, LED_SMD:LED_0603_1608Metric_Pad1.05x0.95mm_HandSolder, symbol Device:LED_Small
- removed D2: RED, LED_SMD:LED_0603_1608Metric_Pad1.05x0.95mm_HandSolder, symbol Device:LED_Small
- removed D3: Yellow, LED_SMD:LED_0603_1608Metric_Pad1.05x0.95mm_HandSolder, symbol Device:LED_Small
- removed D4: BLUE, LED_SMD:LED_0603_1608Metric_Pad1.05x0.95mm_HandSolder, symbol Device:LED_Small
- removed D5: WHITE, LED_SMD:LED_0603_1608Metric_Pad1.05x0.95mm_HandSolder, symbol Device:LED_Small
- removed D6: GREEN, LED_SMD:LED_0603_1608Metric_Pad1.05x0.95mm_HandSolder, symbol Device:LED_Small
- removed R2, R3, R4, R5, R6, R7: 3.3k, Resistor_SMD:R_0603_1608Metric_Pad0.98x0.95mm_HandSolder, symbol Device:R_Small
- added JP501, JP502, JP503, JP504, JP505, JP506, JP507, JP508, JP509, JP510, JP511, JP512, JP513, JP514, JP515, JP516, JP517, JP518, JP519, JP520, JP521, JP522, JP523, JP524, JP525, JP526, JP527, JP528, JP529, JP530, JP531, JP532, JP533, JP534, JP535, JP536, JP537, JP538, JP539, JP540, JP541: SolderJumper_2_Open, symbol Jumper:SolderJumper_2_Open
Connections:
- net DRIVER_1_FWD: now also JP536.2 (B); no longer IC4.17 (PB0)
- net DRIVER_1_REV: now also JP537.2 (B); no longer IC4.18 (PB1)
- net DRIVER_2_FWD: now also JP539.2 (B); no longer IC4.22 (PB10)
- net DRIVER_2_REV: now also JP540.2 (B); no longer IC4.24 (PB11)
- net LIDAR_M_CTR: now also JP504.1 (A); no longer IC4.8 (PA0)
- net LIDAR_RX: now also JP502.1 (A); no longer IC4.11 (PA3)
- net LIDAR_TX: now also JP503.1 (A); no longer IC4.10 (PA2)
- net NRST: now also JP505.1 (A); no longer IC4.7 (PG10-NRST)
- net ODOM2_PHASEA: now also JP518.2 (B); no longer IC4.39 (PC10)
- net ODOM2_PHASEB: now also JP529.1 (A); no longer IC4.38 (PA15)
- net OSC_IN: now also JP507.1 (A); no longer IC4.5 (PF0-OSC_IN)
- net OSC_OUT: now also JP506.1 (A); no longer C7.2, IC4.6 (PF1-OSC_OUT), R1.2, Y1.1
- net STLINK_SWCLK: now also JP520.2 (B); no longer IC4.37 (PA14)
- net STLINK_SWDIO: now also JP522.1 (A); no longer IC4.36 (PA13)
- net STLINK_SWO: now also JP516.2 (B); no longer IC4.41 (PB3)
- net VCP_RX: now also JP526.1 (A); no longer IC4.31 (PA9)
- net VCP_TX: now also JP525.1 (A); no longer IC4.32 (PA10)
- net at IC4.12 (PA4): now also JP541.2 (B)
- net at IC4.2 (PC13): now also JP510.2 (B)
- net at IC4.25 (PB12): now also JP532.2 (B)
- net at IC4.26 (PB13): now also JP531.2 (B)
- net at IC4.27 (PB14): now also JP530.2 (B)
- net at IC4.28 (PB15): now also JP529.2 (B)
- net at IC4.29 (PC6): now also JP528.2 (B)
- net at IC4.3 (PC14-OSC32_IN): now also JP509.2 (B)
- net at IC4.33 (PA11): now also JP524.2 (B)
- net at IC4.34 (PA12): now also JP523.2 (B)
- net at IC4.4 (PC15-OSC32_OUT): now also JP508.2 (B)
- net at IC4.47 (PB9): now also JP521.1 (A)
- net at IC4.9 (PA1): now also JP511.2 (B)
- net IMU_INT1: no longer names the net of IC4.16 (PC4)
- net IMU_INT1: now also JP535.1 (A)
- net IMU_INT2: no longer names the net of IC4.19 (PB2)
- net IMU_INT2: now also JP538.1 (A)
- net IMU_MISO/SDO: no longer names the net of IC4.14 (PA6)
- net IMU_MISO/SDO: now also JP533.1 (A)
- net IMU_MOSI/SDIO: no longer names the net of IC4.15 (PA7)
- net IMU_MOSI/SDIO: now also JP534.1 (A)
- net IMU_SCLK: no longer names the net of IC4.13 (PA5)
- net IMU_SCLK: now also JP501.1 (A)
- net ODOM_PHASEA: no longer names the net of IC4.45 (PB7)
- net ODOM_PHASEA: now also JP512.1 (A)
- net ODOM_PHASEB: no longer names the net of IC4.44 (PB6)
- net ODOM_PHASEB: now also JP513.1 (A)
- net TOF_GPIO1: no longer names the net of IC4.43 (PB5)
- net TOF_GPIO1: now also JP514.1 (A)
- net TOF_SCL: no longer names the net of IC4.30 (PA8)
- net TOF_SCL: now also JP527.2 (B)
- net TOF_SDA: no longer names the net of IC4.40 (PC11)
- net TOF_SDA: now also JP517.1 (A)
- net TOF_XSHUT: no longer names the net of IC4.42 (PB4)
- net TOF_XSHUT: now also JP515.1 (A)
- new net: C7.2, R1.2, Y1.1
- new net: IC4.36 (PA13), JP522.2 (B)
- new net: IC4.11 (PA3), JP502.2 (B)
- new net: IC4.24 (PB11), JP540.1 (A)
- new net: IC4.31 (PA9), JP526.2 (B)
- new net: IC4.5 (PF0-OSC_IN), JP507.2 (B)
- new net: IC4.8 (PA0), JP504.2 (B)
- new net: IC4.32 (PA10), JP525.2 (B)
- new net: IC4.39 (PC10), JP518.1 (A)
- new net: IC4.38 (PA15), JP519.1 (A)
- new net: IC4.37 (PA14), JP520.1 (A)
- new net: IC4.17 (PB0), JP536.1 (A)
- new net: IC4.18 (PB1), JP537.1 (A)
- new net: IC4.6 (PF1-OSC_OUT), JP506.2 (B)
- new net: IC4.10 (PA2), JP503.2 (B)
- new net: IC4.22 (PB10), JP539.1 (A)
- new net: IC4.41 (PB3), JP516.1 (A)
- new net: IC4.7 (PG10-NRST), JP505.2 (B)
- new net CC1: JP513.2 (B)
- new net CC2: JP515.2 (B)
- new net EXPANDER_EXTI: JP524.1 (A)
- new net I2C_MAIN_SCL: JP527.1 (A)
- new net I2C_MAIN_SDA: JP517.2 (B)
- new net IMU_SCL: JP519.2 (B)
- new net IMU_SDA: JP512.2 (B)
- new net ODOM1_PHASEA: JP528.1 (A)
- new net ODOM1_PHASEB: JP514.2 (B)
- no-connect marks 17 -> 19
Other:
- note removed: "4 LEDs for debbuging"
- note removed: "LEDs"

Commit message: KiCAD V3 - 18.09.2024
Connections:
- net BUTTON_1: now also SW4.1; no longer SW2.1
- net BUTTON_3: now also SW2.1; no longer SW4.1
- net MOUSTACHE_3: now reaches JP534.2 (B)
- net MOUSTACHE_4: now reaches JP535.2 (B)
- net MOUSTACHE_2: now reaches JP533.2 (B)
- net MOUSTACHE_1: now reaches JP538.2 (B)
- net DAC-: now reaches JP501.2 (B)
- net DAC+: now reaches JP541.1 (A)
- no-connect marks 19 -> 13
Changed lines of the file:
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@@
 	)
 	(no_connect
-		(at 59.69 125.73)
-	)
-	(no_connect
 		(at 246.38 53.34)
 	)
@@
 	)
 	(no_connect
-		(at 54.61 125.73)
-	)
-	(no_connect
-		(at 52.07 125.73)
-	)
-	(no_connect
-		(at 57.15 125.73)
-	)
-	(no_connect
 		(at 97.79 95.25)
 	)
@@
 	)
 	(no_connect
-		(at 67.31 125.73)
-	)
-	(no_connect
 		(at 97.79 100.33)
 	)
@@
 		(at 97.79 97.79)
 	)
-	(no_connect
-		(at 36.83 100.33)
-	)
 	(wire
 		(pts
@@
 		)
 	)
-	(label "BUTTON_2"
-		(at 140.97 123.19 0)
-		(fields_autoplaced yes)
-		(effects
-			(font
-				(size 1.27 1.27)
-				(bold yes)
-			)
-			(justify left bottom)
-		)
-	)
 	(label "NRST"
 		(at 139.7 97.79 0)
@@
 		)
 	)
-	(label "BUTTON_3"
-		(at 140.97 129.54 0)
+	(label "VREF"
+		(at 104.14 163.83 0)
 		(fields_autoplaced yes)
 		(effects
@@
 		)
 	)
-	(label "VREF"
-		(at 104.14 163.83 0)
+	(label "STLINK_SWCLK"
+		(at 250.19 48.26 0)
 		(fields_autoplaced yes)
 		(effects
@@
 		)
 	)
-	(label "BUTTON_1"
-		(at 140.97 116.84 0)
+	(label "VCP_RX"
+		(at 97.79 86.36 0)
 		(fields_autoplaced yes)
 		(effects
 			(font
 				(size 1.27 1.27)
+				(thickness 0.254)
 				(bold yes)
 			)
@@
 		)
 	)
-	(label "STLINK_SWCLK"
-		(at 250.19 48.26 0)
+	(label "NRST"
+		(at 250.19 55.88 0)
 		(fields_autoplaced yes)
 		(effects
@@
 		)
 	)
-	(label "VCP_RX"
-		(at 97.79 86.36 0)
+	(label "OSC_OUT"
+		(at 135.89 52.07 0)
 		(fields_autoplaced yes)
 		(effects
 			(font
 				(size 1.27 1.27)
-				(thickness 0.254)
 				(bold yes)
 			)
@@
 		)
 	)
-	(label "NRST"
-		(at 250.19 55.88 0)
+	(label "STLINK_SWDIO"
+		(at 97.79 73.66 0)
 		(fields_autoplaced yes)
 		(effects
 			(font
 				(size 1.27 1.27)
+				(thickness 0.254)
 				(bold yes)
 			)
@@
 		)
 	)
-	(label "OSC_OUT"
-		(at 135.89 52.07 0)
+	(global_label "BUTTON_2"
+		(shape input)
+		(at 140.97 123.19 180)
 		(fields_autoplaced yes)
 		(effects
@@
 				(bold yes)
 			)
-			(justify left bottom)
+			(justify right)
+		)
+		(property "Intersheetrefs" "${INTERSHEET_REFS}"
+			(at 128.135 123.19 0)
+			(effects
+				(font
+					(size 1.27 1.27)
+				)
+				(justify right)
+				(hide yes)
+			)
 		)
 	)
-	(label "STLINK_SWDIO"
-		(at 97.79 73.66 0)
+	(global_label "BUTTON_1"
+		(shape input)
+		(at 140.97 129.54 180)
 		(fields_autoplaced yes)
 		(effects
 			(font
 				(size 1.27 1.27)
-				(thickness 0.254)
 				(bold yes)
 			)
-			(justify left bottom)
+			(justify right)
+		)
+		(property "Intersheetrefs" "${INTERSHEET_REFS}"
+			(at 128.135 129.54 0)
+			(effects
+				(font
+					(size 1.27 1.27)
+				)
+				(justify right)
+				(hide yes)
+			)
+		)
+	)
+	(global_label "BUTTON_3"
+		(shape input)
+		(at 140.97 116.84 180)
+		(fields_autoplaced yes)
+		(effects
+			(font
+				(size 1.27 1.27)
+				(bold yes)
+			)
+			(justify right)
+		)
+		(property "Intersheetrefs" "${INTERSHEET_REFS}"
+			(at 128.135 116.84 0)
+			(effects
+				(font
+					(size 1.27 1.27)
+				)
+				(justify right)
+				(hide yes)
+			)
 		)
 	)
@@
 		)
 	)
+	(hierarchical_label "DAC-"
+		(shape input)
+		(at 52.07 125.73 270)
+		(fields_autoplaced yes)
+		(effects
+			(font
+				(size 1.27 1.27)
+				(thickness 0.254)
+				(bold yes)
+			)
+			(justify right)
+		)
+	)
 	(hierarchical_label "DRIVER_2_FWD"
 		(shape input)
@@
 		)
 	)
+	(hierarchical_label "DAC+"
+		(shape input)
+		(at 36.83 100.33 180)
+		(fields_autoplaced yes)
+		(effects
+			(font
+				(size 1.27 1.27)
+				(thickness 0.254)
+				(bold yes)
+			)
+			(justify right)
+		)
+	)
 	(hierarchical_label "I2C_MAIN_SDA"
 		(shape input)
@@
 		)
 	)
+	(hierarchical_label "MOUSTACHE_1"
+		(shape input)
+		(at 67.31 125.73 270)
+		(fields_autoplaced yes)
+		(effects
+			(font
+				(size 1.27 1.27)
+				(thickness 0.254)
+				(bold yes)
+			)
+			(justify right)
+		)
+	)
 	(hierarchical_label "ODOM1_PHASEA"
 		(shape input)
@@
 		)
 	)
+	(hierarchical_label "MOUSTACHE_3"
+		(shape input)
+		(at 57.15 125.73 270)
+		(fields_autoplaced yes)
+		(effects
+			(font
+				(size 1.27 1.27)
+				(thickness 0.254)
+				(bold yes)
+			)
+			(justify right)
+		)
+	)
 	(hierarchical_label "LIDAR_RX"
 		(shape input)
@@
 		)
 	)
+	(hierarchical_label "MOUSTACHE_2"
+		(shape input)
+		(at 54.61 125.73 270)
+		(fields_autoplaced yes)
+		(effects
+			(font
+				(size 1.27 1.27)
+				(thickness 0.254)
+				(bold yes)
+			)
+			(justify right)
+		)
+	)
+	(hierarchical_label "MOUSTACHE_4"
+		(shape input)
+		(at 59.69 125.73 270)
+		(fields_autoplaced yes)
+		(effects
+			(font
+				(size 1.27 1.27)
+				(thickness 0.254)
+				(bold yes)
+			)
+			(justify right)
+		)
+	)
 	(hierarchical_label "CC1"
 		(shape input)
@@
 					(reference "IC4")
 					(unit 1)
+				)
+				(path "/d6e3fbeb-d028-494d-83bf-2e4a8b12578d/ac7f7f04-c418-4551-b204-a999b9c3c440/d8c0a3ec-14ca-4cad-91fd-ac8f1e686c9a"
+					(reference "IC4")
+					(unit 1)

Commit message: STM32 KiCAD V4 - 20.09.2024
Connections:
- net MOUSTACHE_1: now also JP530.1 (A); no longer JP538.2 (B)
- net MOUSTACHE_2: now also JP531.1 (A); no longer JP533.2 (B)
- net MOUSTACHE_3: now also JP535.2 (B); no longer JP534.2 (B)
- net MOUSTACHE_4: now also JP538.2 (B); no longer JP535.2 (B)
- new net ASSERV1_OUT: JP533.2 (B)
- new net ASSERV2_OUT: JP534.2 (B)
- no-connect marks 13 -> 11
Changed lines of the file:
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@@
-	)
-	(no_connect
-		(at 97.79 95.25)
 	)
 	(no_connect
@@
 	(no_connect
 		(at 36.83 74.93)
-	)
-	(no_connect
-		(at 97.79 97.79)
 	)
 	(wire
@@
 		)
 	)
+	(hierarchical_label "MOUSTACHE_1"
+		(shape input)
+		(at 97.79 95.25 0)
+		(fields_autoplaced yes)
+		(effects
+			(font
+				(size 1.27 1.27)
+				(thickness 0.254)
+				(bold yes)
+			)
+			(justify left)
+		)
+	)
 	(hierarchical_label "IMU_SCL"
 		(shape input)
@@
 		)
 	)
-	(hierarchical_label "MOUSTACHE_1"
+	(hierarchical_label "MOUSTACHE_4"
 		(shape input)
 		(at 67.31 125.73 270)
@@
 		)
 	)
+	(hierarchical_label "ASSERV2_OUT"
+		(shape input)
+		(at 57.15 125.73 270)
+		(fields_autoplaced yes)
+		(effects
+			(font
+				(size 1.27 1.27)
+				(thickness 0.254)
+				(bold yes)
+			)
+			(justify right)
+		)
+	)
+	(hierarchical_label "LIDAR_RX"
+		(shape input)
+		(at 36.83 97.79 180)
+		(fields_autoplaced yes)
+		(effects
+			(font
+				(size 1.27 1.27)
+				(thickness 0.254)
+				(bold yes)
+			)
+			(justify right)
+		)
+	)
+	(hierarchical_label "I2C_MAIN_SCL"
+		(shape input)
+		(at 97.79 87.63 0)
+		(fields_autoplaced yes)
+		(effects
+			(font
+				(size 1.27 1.27)
+				(thickness 0.254)
+				(bold yes)
+			)
+			(justify left)
+		)
+	)
+	(hierarchical_label "ASSERV1_OUT"
+		(shape input)
+		(at 54.61 125.73 270)
+		(fields_autoplaced yes)
+		(effects
+			(font
+				(size 1.27 1.27)
+				(thickness 0.254)
+				(bold yes)
+			)
+			(justify right)
+		)
+	)
 	(hierarchical_label "MOUSTACHE_3"
 		(shape input)
-		(at 57.15 125.73 270)
+		(at 59.69 125.73 270)
 		(fields_autoplaced yes)
 		(effects
@@
 		)
 	)
-	(hierarchical_label "LIDAR_RX"
-		(shape input)
-		(at 36.83 97.79 180)
-		(fields_autoplaced yes)
-		(effects
-			(font
-				(size 1.27 1.27)
-				(thickness 0.254)
-				(bold yes)
-			)
-			(justify right)
-		)
-	)
-	(hierarchical_label "I2C_MAIN_SCL"
-		(shape input)
-		(at 97.79 87.63 0)
+	(hierarchical_label "CC1"
+		(shape input)
+		(at 64.77 41.91 90)
 		(fields_autoplaced yes)
 		(effects
@@
 	(hierarchical_label "MOUSTACHE_2"
 		(shape input)
-		(at 54.61 125.73 270)
-		(fields_autoplaced yes)
-		(effects
-			(font
-				(size 1.27 1.27)
-				(thickness 0.254)
-				(bold yes)
-			)
-			(justify right)
-		)
-	)
-	(hierarchical_label "MOUSTACHE_4"
-		(shape input)
-		(at 59.69 125.73 270)
-		(fields_autoplaced yes)
-		(effects
-			(font
-				(size 1.27 1.27)
-				(thickness 0.254)
-				(bold yes)
-			)
-			(justify right)
-		)
-	)
-	(hierarchical_label "CC1"
-		(shape input)
-		(at 64.77 41.91 90)
-		(fields_autoplaced yes)
-		(effects
+		(at 97.79 97.79 0)
+		(fields_autoplaced yes)
+		(effects

Commit message: STM32 KiCAD V5 - 20.09.2024
Other:
- note added: "STLink-V3"
- note added: "voir STDC14"
- note removed: "STlink"
- note removed: "mauvaise ref de composant voir STDC14"
- moved on the sheet: C1, C2, C3, C4, C5, IC4, JP501, JP502, JP503, JP504, JP505, JP506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
