File: electronique/schematic_draft/tom&Jerry_Draft/tom&Jerry_Draft.kicad_pcb (KiCad board)
At the start: 4 copper layers, 54 x 57 mm, 173 parts, among them IC1401 NCS199A2RSQT2G, IC1501 NCS199A2RSQT2G, IC301 TCA9555RTWR, J1701 Conn_01x02, J1801 Conn_01x02, J1901 Conn_01x02, J2001 Conn_01x02, J201 Interrupteur, J202 USB_C_Receptacle_USB2.0_16P, J203 Conn_01x02, J204 Conn_01x02, J301 Conn_01x08, J401 Conn_01x06, J402 Conn_01x06, J501 Conn_ST_STDC14, J601 Conn_01x03, SW501 SW_Push, SW502 SW_Push, SW503 SW_Push, U1301 LP5812ADSDR, U1401 ZXBM5210-S, U1501 ZXBM5210-S, U201 MP1475DJ-LF-P, U202 BQ25172DSGR, U301 ADXL343, U501 STM32G431CBU6, U601 PAM8302AAY, Y501 16MHz

Commit message: Changing footprint V0.2
Parts:
- added D201: D, Tom&Jerry:SODFL4825X110N, F.Cu at (186.4, 54.5)
- added D202: D, Tom&Jerry:SODFL4825X110N, F.Cu at (186.4, 58.5)
- added J1001: Conn_02x05_Odd_FEMALE, Connector_PinSocket_1.27mm:PinSocket_2x05_P1.27mm_Vertical, F.Cu at (183.0, 33.4)
- added J1101: Conn_02x05_Odd_FEMALE, Connector_PinSocket_1.27mm:PinSocket_2x05_P1.27mm_Vertical, F.Cu at (102.9, 86.3)
- added J1201: Conn_02x05_Odd_FEMALE, Connector_PinSocket_1.27mm:PinSocket_2x05_P1.27mm_Vertical, F.Cu at (108.9, 97.5)
- added J701: Conn_02x05_Odd_FEMALE, Connector_PinSocket_1.27mm:PinSocket_2x05_P1.27mm_Vertical, F.Cu at (175.9, 33.4)
- added J801: Conn_02x05_Odd_FEMALE, Connector_PinSocket_1.27mm:PinSocket_2x05_P1.27mm_Vertical, F.Cu at (183.0, 23.0)
- added J901: Conn_02x05_Odd_FEMALE, Connector_PinSocket_1.27mm:PinSocket_2x05_P1.27mm_Vertical, F.Cu at (175.9, 23.0)
- C208: footprint Tom&Jerry:PQFN80P300X500X100-14N -> Tom&Jerry:CAPAE1350X1400N
- moved C501 180.1 mm to (259.6, 29.7)
- moved C502 180.1 mm to (259.6, 31.7)
- moved C504 180.1 mm to (259.6, 33.7)
- moved C506 180.1 mm to (259.6, 35.7)
- moved C507 180.1 mm to (259.6, 37.6)
- moved C508 180.1 mm to (259.6, 39.6)
- moved C509 180.1 mm to (262.5, 29.7)
- moved C510 180.1 mm to (262.5, 31.7)
- moved C511 180.1 mm to (262.5, 33.7)
- moved C512 180.1 mm to (262.5, 35.7)
- moved C514 180.1 mm to (262.5, 37.6)
- moved IC1401 180.1 mm to (269.1, 73.1)
- moved U1501 180.1 mm to (256.5, 68.0)
- moved C1001 180.1 mm to (219.1, 103.6)
- moved C1101 180.1 mm to (219.1, 90.6)
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
Commit message: Ajout des bonnes empreintes
Parts:
- removed C1001, C1101, C1201, C1401, C1501, C401, C507, C701, C801, C901: 100nF, Capacitor_SMD:C_0402_1005Metric
- removed C1002, C1102, C1202, C702, C802, C902: 4.7uF, Capacitor_SMD:C_0603_1608Metric
- removed C1402, C1404, C1405, C1502, C1504, C1505: 1uF, Capacitor_SMD:C_0603_1608Metric
- removed C1403, C1503: 10uF, Capacitor_SMD:C_0603_1608Metric
- removed C1701, C1801, C1901, C2001, C207, C211, C502, C506, C508, C509: 10n, Capacitor_SMD:C_0402_1005Metric
- removed C201, C203, C204: 22uF, Capacitor_SMD:C_0805_2012Metric
- removed C202: 0.1u, Capacitor_SMD:C_0402_1005Metric
- removed C205, C209: 0.1uF, Capacitor_SMD:C_0402_1005Metric
- removed C206, C510, C511, C512, C514, C605: 100n, Capacitor_SMD:C_0402_1005Metric
- removed C208: 1mF, Tom&Jerry:CAPAE1350X1400N
- removed C210: 15pF, Capacitor_SMD:C_0402_1005Metric
- removed C212, C213, C503, C505, C602, C604: 1u, Capacitor_SMD:C_0603_1608Metric
- removed C301: 100n, Capacitor_SMD:C_0805_2012Metric
- removed C501, C504: 10p, Capacitor_SMD:C_0402_1005Metric
- removed C513: 4.7u, Capacitor_SMD:C_0603_1608Metric
- removed C601: 10u, Capacitor_SMD:C_0603_1608Metric
- removed C603, C606: 220p, Capacitor_SMD:C_0402_1005Metric
- removed D201, D202: D, Tom&Jerry:SODFL4825X110N
- removed D203, D204, D205, D206, D207: LED, LED_SMD:LED_0603_1608Metric_Pad1.05x0.95mm_HandSolder
- removed FB601, FB602: FerriteBead_Small, Inductor_SMD:L_0805_2012Metric
- removed IC1401, IC1501: NCS199A2RSQT2G, Tom&Jerry:SOT65P210X110-6N
- removed IC301: TCA9555RTWR, Tom&Jerry:RTW24_2P45X2P45
- removed J1001, J1101, J1201, J701, J801, J901: Conn_02x05_Odd_FEMALE, Connector_PinSocket_1.27mm:PinSocket_2x05_P1.27mm_Vertical
- removed J1701, J1801, J1901, J2001, J203, J204: Conn_01x02, Connector_JST:JST_XH_S2B-XH-A-1_1x02_P2.50mm_Horizontal
- removed J201: Interrupteur, Tom&Jerry:Switch-3
- removed J202: USB_C_Receptacle_USB2.0_16P, Connector_USB:USB_C_Receptacle_HRO_TYPE-C-31-M-12
- removed J301: Conn_01x08, Connector_JST:JST_XH_S8B-XH-A_1x08_P2.50mm_Horizontal
- removed J401, J402: Conn_01x06, Connector_JST:JST_XH_S6B-XH-A_1x06_P2.50mm_Horizontal
- removed J501: Conn_ST_STDC14, Connector_PinHeader_1.27mm:PinHeader_2x07_P1.27mm_Vertical_SMD
- removed J601: Conn_01x03, Connector_JST:JST_XH_S3B-XH-A_1x03_P2.50mm_Horizontal
- removed JP201, JP202, JP203, JP204: SolderJumper_2_Open, Jumper:SolderJumper-2_P1.3mm_Open_TrianglePad1.0x1.5mm
- removed L201: 4.7uH, Inductor_SMD:L_0603_1608Metric_Pad1.05x0.95mm_HandSolder
- removed L501: 39n, Inductor_SMD:L_0603_1608Metric_Pad1.05x0.95mm_HandSolder
- removed L502: 47n, Inductor_SMD:L_0603_1608Metric_Pad1.05x0.95mm_HandSolder
- removed L503: 6u, Inductor_SMD:L_0603_1608Metric_Pad1.05x0.95mm_HandSolder
- removed LED1301, LED1302, LED1303, LED1304: RGB, Tom&Jerry:5988G10313F
- removed PS201: BU33SD5WG-TR, Tom&Jerry:SOT95P280X125-5N
- removed R101, R102, R103, R104, R1701, R1702, R1801, R1802, R1901, R1902, R2001, R2002, R213, R503, R504, R505, R506: 10k, Resistor_SMD:R_0402_1005Metric
- removed R1401, R1501: 0.015, Resistor_SMD:R_0402_1005Metric
- removed R201: 20, Resistor_SMD:R_0402_1005Metric
- removed R202: 100m, Resistor_SMD:R_0402_1005Metric
- removed R203, R204, R401, R402, R502: 100k, Resistor_SMD:R_0402_1005Metric
- removed R205: 16k, Resistor_SMD:R_0402_1005Metric
- removed R206: 40.2k, Resistor_SMD:R_0402_1005Metric
- removed R207: 7.68k, Resistor_SMD:R_0402_1005Metric
- removed R208: 15k, Resistor_SMD:R_0402_1005Metric
- removed R209: R_Small, Resistor_SMD:R_0402_1005Metric
- removed R210: 3.6k, Resistor_SMD:R_0402_1005Metric
- removed R211, R212: 27k, Resistor_SMD:R_0402_1005Metric
- removed R214, R215, R216, R217: 3.3k, Resistor_SMD:R_0402_1005Metric
- removed R501: 10R, Resistor_SMD:R_0402_1005Metric
- removed SW501, SW502, SW503: SW_Push, Button_Switch_SMD:SW_Push_1P1T_NO_6x6mm_H9.5mm
- removed TP201, TP202, TP203, TP204: TestPoint_Small, Test_Point:TestPoint_Pad_D1.5mm
- removed TP501: PA0, Test_Point:TestPoint_Pad_D1.5mm
- removed TP502: PA1, Test_Point:TestPoint_Pad_D1.5mm
- removed TP503: PA4, Test_Point:TestPoint_Pad_D1.5mm
- removed TP504: PA6, Test_Point:TestPoint_Pad_D1.5mm
- removed TP505: PA7, Test_Point:TestPoint_Pad_D1.5mm
- removed TP506: PC6, Test_Point:TestPoint_Pad_D1.5mm
- removed TP507: PA9, Test_Point:TestPoint_Pad_D1.5mm
- removed TP508: PA10, Test_Point:TestPoint_Pad_D1.5mm
- removed TP509: PA11, Test_Point:TestPoint_Pad_D1.5mm
- removed TP510: PA12, Test_Point:TestPoint_Pad_D1.5mm
- removed TP511: PB0, Test_Point:TestPoint_Pad_D1.5mm
- removed TP512: PB1, Test_Point:TestPoint_Pad_D1.5mm
- removed TP513: PB4, Test_Point:TestPoint_Pad_D1.5mm
- removed TP514: PB5, Test_Point:TestPoint_Pad_D1.5mm
- removed TP515: PB6, Test_Point:TestPoint_Pad_D1.5mm
- removed TP516: PB10, Test_Point:TestPoint_Pad_D1.5mm
- removed TP517: PB11, Test_Point:TestPoint_Pad_D1.5mm
- removed U1301: LP5812ADSDR, Tom&Jerry:WSON8_DSD_TEX
- removed U1401, U1501: ZXBM5210-S, Tom&Jerry:SOIC127P600X175-8N
- removed U201: MP1475DJ-LF-P, Tom&Jerry:SOT65P280X100-8N
- removed U202: BQ25172DSGR, Tom&Jerry:IC_BQ25172DSGR
- removed U301: ADXL343, Tom&Jerry:PQFN80P300X500X100-14N
- removed U501: STM32G431CBU6, Package_DFN_QFN:QFN-48-1EP_7x7mm_P0.5mm_EP5.1x5.1mm
- removed U601: PAM8302AAY, Tom&Jerry:DFN300X300X80-8N
- removed Y501: 16MHz, Crystal:Crystal_SMD_3225-4Pin_3.2x2.5mm

Commit message: Ajout V2 TOF + MultiPCB Panalize
Parts:
- added C1001: 1uF, Capacitor_SMD:C_0603_1608Metric, F.Cu at (256.6, 99.8)
- added C1002: 1uF, Capacitor_SMD:C_0603_1608Metric, F.Cu at (256.6, 102.3)
- added C1003: 1uF, Capacitor_SMD:C_0603_1608Metric, F.Cu at (256.6, 104.8)
- added C1004: 10uF, Capacitor_SMD:C_0603_1608Metric, F.Cu at (256.6, 107.4)
- added C1005: 100nF, Capacitor_SMD:C_0402_1005Metric, F.Cu at (264.7, 108.0)
- added C1201: 10n, Capacitor_SMD:C_0402_1005Metric, F.Cu at (265.5, 85.6)
- added C1301: 10n, Capacitor_SMD:C_0402_1005Metric, F.Cu at (205.9, 119.9)
- added C1401: 10n, Capacitor_SMD:C_0402_1005Metric, F.Cu at (191.5, 119.9)
- added C1501: 10n, Capacitor_SMD:C_0402_1005Metric, F.Cu at (265.5, 116.0)
- added C1601: 100nF, Capacitor_SMD:C_0402_1005Metric, F.Cu at (242.8, 108.0)
- added C1602: 4.7uF, Capacitor_SMD:C_0603_1608Metric, F.Cu at (239.3, 108.2)
- added C1603: 100nF, Capacitor_SMD:C_0402_1005Metric, F.Cu at (242.8, 109.9)
- added C1604: 4.7uF, Capacitor_SMD:C_0603_1608Metric, F.Cu at (239.3, 110.7)
- added C1605: 100nF, Capacitor_SMD:C_0402_1005Metric, F.Cu at (242.8, 111.9)
- added C1606: 4.7uF, Capacitor_SMD:C_0603_1608Metric, F.Cu at (239.3, 113.2)
- added C201: 22uF, Capacitor_SMD:C_0805_2012Metric, F.Cu at (212.1, 67.2)
- added C202: 0.1uF, Capacitor_SMD:C_0402_1005Metric, F.Cu at (218.9, 39.0)
- added C203: 1u, Capacitor_SMD:C_0603_1608Metric, F.Cu at (216.3, 71.4)
- added C204: 0.1u, Capacitor_SMD:C_0402_1005Metric, F.Cu at (218.9, 41.0)
- added C205: 0.1uF, Capacitor_SMD:C_0402_1005Metric, F.Cu at (218.9, 42.9)
- added C206: 15pF, Capacitor_SMD:C_0402_1005Metric, F.Cu at (218.9, 44.9)
- added C207: 22uF, Capacitor_SMD:C_0805_2012Metric, F.Cu at (212.1, 70.2)
- added C208: 1u, Capacitor_SMD:C_0603_1608Metric, F.Cu at (216.3, 73.9)
- added C209: 22uF, Capacitor_SMD:C_0805_2012Metric, F.Cu at (212.1, 73.2)
- added C210: 100n, Capacitor_SMD:C_0402_1005Metric, F.Cu at (218.9, 46.9)
- added C211: 10n, Capacitor_SMD:C_0402_1005Metric, F.Cu at (218.9, 48.8)
- added C212: 10n, Capacitor_SMD:C_0402_1005Metric, F.Cu at (218.9, 50.8)
- added C213: 1mF, Tom&Jerry:CAPAE1350X1400N, F.Cu at (189.6, 45.9)
- added C301: 100n, Capacitor_SMD:C_0805_2012Metric, F.Cu at (233.0, 66.4)
- added C401: 100nF, Capacitor_SMD:C_0402_1005Metric, F.Cu at (233.9, 85.6)
- added C501: 100n, Capacitor_SMD:C_0402_1005Metric, F.Cu at (206.7, 81.6)
- added C502: 1u, Capacitor_SMD:C_0603_1608Metric, F.Cu at (204.3, 93.8)
- added C503: 100n, Capacitor_SMD:C_0402_1005Metric, F.Cu at (206.7, 83.6)
- added C504: 10n, Capacitor_SMD:C_0402_1005Metric, F.Cu at (206.7, 85.6)
- added C505: 100n, Capacitor_SMD:C_0402_1005Metric, F.Cu at (206.7, 87.5)
- added C506: 4.7u, Capacitor_SMD:C_0603_1608Metric, F.Cu at (204.3, 96.3)
- added C507: 10n, Capacitor_SMD:C_0402_1005Metric, F.Cu at (206.7, 89.5)
- added C508: 1u, Capacitor_SMD:C_0603_1608Metric, F.Cu at (204.3, 98.9)
- added C509: 100n, Capacitor_SMD:C_0402_1005Metric, F.Cu at (206.7, 91.5)
- added C510: 10p, Capacitor_SMD:C_0402_1005Metric, F.Cu at (209.5, 81.6)
- added C511: 10p, Capacitor_SMD:C_0402_1005Metric, F.Cu at (209.5, 83.6)
- added C512: 10n, Capacitor_SMD:C_0402_1005Metric, F.Cu at (209.5, 85.6)
- added C513: 100nF, Capacitor_SMD:C_0402_1005Metric, F.Cu at (209.5, 87.5)
- added C514: 10n, Capacitor_SMD:C_0402_1005Metric, F.Cu at (209.5, 89.5)
- added C601: 1u, Capacitor_SMD:C_0603_1608Metric, F.Cu at (226.9, 111.0)
- added C602: 10u, Capacitor_SMD:C_0603_1608Metric, F.Cu at (226.9, 113.5)
- added C603: 100n, Capacitor_SMD:C_0402_1005Metric, F.Cu at (226.4, 118.3)
- added C604: 1u, Capacitor_SMD:C_0603_1608Metric, F.Cu at (226.9, 116.0)
- added C605: 220p, Capacitor_SMD:C_0402_1005Metric, F.Cu at (226.4, 120.2)
- added C606: 220p, Capacitor_SMD:C_0402_1005Metric, F.Cu at (226.4, 122.2)
- added C701: 100nF, Capacitor_SMD:C_0402_1005Metric, F.Cu at (242.8, 90.0)
- added C702: 4.7uF, Capacitor_SMD:C_0603_1608Metric, F.Cu at (239.3, 90.3)
- added C703: 100nF, Capacitor_SMD:C_0402_1005Metric, F.Cu at (242.8, 92.0)
- added C704: 4.7uF, Capacitor_SMD:C_0603_1608Metric, F.Cu at (239.3, 92.8)
- added C705: 100nF, Capacitor_SMD:C_0402_1005Metric, F.Cu at (242.8, 94.0)
- added C706: 4.7uF, Capacitor_SMD:C_0603_1608Metric, F.Cu at (239.3, 95.3)
- added C901: 1uF, Capacitor_SMD:C_0603_1608Metric, F.Cu at (239.3, 117.8)
- added C902: 1uF, Capacitor_SMD:C_0603_1608Metric, F.Cu at (239.3, 120.3)
- added C903: 1uF, Capacitor_SMD:C_0603_1608Metric, F.Cu at (239.3, 122.8)
- added C904: 10uF, Capacitor_SMD:C_0603_1608Metric, F.Cu at (239.3, 125.3)
- added C905: 100nF, Capacitor_SMD:C_0402_1005Metric, F.Cu at (247.4, 126.0)
- added D201: LED, LED_SMD:LED_0603_1608Metric_Pad1.05x0.95mm_HandSolder, F.Cu at (202.4, 67.0)
- added D202: LED, LED_SMD:LED_0603_1608Metric_Pad1.05x0.95mm_HandSolder, F.Cu at (202.4, 69.6)
- added D203: LED, LED_SMD:LED_0603_1608Metric_Pad1.05x0.95mm_HandSolder, F.Cu at (202.4, 72.2)
- added D204: LED, LED_SMD:LED_0603_1608Metric_Pad1.05x0.95mm_HandSolder, F.Cu at (202.4, 74.8)
- added D205: D, Tom&Jerry:SODFL4825X110N, F.Cu at (212.4, 55.8)
- added D206: D, Tom&Jerry:SODFL4825X110N, F.Cu at (212.4, 59.8)
- added D207: LED, LED_SMD:LED_0603_1608Metric_Pad1.05x0.95mm_HandSolder, F.Cu at (202.4, 77.3)
- added FB601: FerriteBead_Small, Inductor_SMD:L_0805_2012Metric, F.Cu at (221.2, 124.7)
- added FB602: FerriteBead_Small, Inductor_SMD:L_0805_2012Metric, F.Cu at (221.2, 127.4)
- added H1601: MountingHole_Pad, MountingHole:MountingHole_3.2mm_M3_Pad_Via, F.Cu at (29.3, 19.9)
- added H1602: MountingHole_Pad, MountingHole:MountingHole_3.2mm_M3_Pad_Via, F.Cu at (29.3, 27.8)
- added H701: MountingHole_Pad, MountingHole:MountingHole_3.2mm_M3_Pad_Via, F.Cu at (19.4, 19.9)
- added H702: MountingHole_Pad, MountingHole:MountingHole_3.2mm_M3_Pad_Via, F.Cu at (19.4, 27.8)
- added IC1001: NCS199A2RSQT2G, Tom&Jerry:SOT65P210X110-6N, F.Cu at (261.0, 107.0)
- added IC301: TCA9555RTWR, Tom&Jerry:RTW24_2P45X2P45, F.Cu at (234.0, 55.0)
- added IC901: NCS199A2RSQT2G, Tom&Jerry:SOT65P210X110-6N, F.Cu at (243.7, 124.9)
- added J1201: Conn_01x02, Connector_JST:JST_XH_S2B-XH-A-1_1x02_P2.50mm_Horizontal, F.Cu at (258.1, 85.6)
- added J1301: Conn_01x02, Connector_JST:JST_XH_S2B-XH-A-1_1x02_P2.50mm_Horizontal, F.Cu at (198.5, 119.8)
- added J1401: Conn_01x02, Connector_JST:JST_XH_S2B-XH-A-1_1x02_P2.50mm_Horizontal, F.Cu at (184.1, 119.8)
- added J1501: Conn_01x02, Connector_JST:JST_XH_S2B-XH-A-1_1x02_P2.50mm_Horizontal, F.Cu at (258.1, 116.0)
- added J1601: Conn_02x05_Odd_FEMALE, Connector_PinSocket_1.27mm:PinSocket_2x05_P1.27mm_Vertical, F.Cu at (240.5, 100.2)
- added J1602: Conn_02x05_Odd_FEMALE, Connector_PinSocket_1.27mm:PinSocket_2x05_P1.27mm_Vertical, F.Cu at (245.6, 100.2)
- added J1603: Conn_02x05_Odd_FEMALE, Connector_PinSocket_1.27mm:PinSocket_2x05_P1.27mm_Vertical, F.Cu at (250.7, 100.2)
- added J201: Conn_01x02, Connector_JST:JST_XH_S2B-XH-A-1_1x02_P2.50mm_Horizontal, F.Cu at (202.1, 42.9)
- added J202: USB_C_Receptacle_USB2.0_16P, Connector_USB:USB_C_Receptacle_HRO_TYPE-C-31-M-12, F.Cu at (186.5, 67.4)
- added J203: Conn_01x02, Connector_JST:JST_XH_S2B-XH-A-1_1x02_P2.50mm_Horizontal, F.Cu at (211.5, 42.9)
- added J204: Interrupteur, Tom&Jerry:Switch-3, F.Cu at (190.2, 57.6)
- added J301: FTSH-105-01-F-DV-P-TR, Tom&Jerry:SAMTEC_FTSH-105-01-F-DV-P-TR, F.Cu at (226.9, 42.2)
- added J302: FTSH-105-01-F-DV-P-TR, Tom&Jerry:SAMTEC_FTSH-105-01-F-DV-P-TR, F.Cu at (226.9, 50.6)
- added J303: FTSH-105-01-F-DV-P-TR, Tom&Jerry:SAMTEC_FTSH-105-01-F-DV-P-TR, F.Cu at (226.9, 59.0)
- added J304: FTSH-105-01-F-DV-P-TR, Tom&Jerry:SAMTEC_FTSH-105-01-F-DV-P-TR, F.Cu at (226.9, 67.4)
- added J305: Conn_01x08, Connector_JST:JST_XH_S8B-XH-A_1x08_P2.50mm_Horizontal, F.Cu at (234.3, 41.3)
- added J401: Conn_01x06, Connector_JST:JST_XH_S6B-XH-A_1x06_P2.50mm_Horizontal, F.Cu at (216.4, 84.0)
- added J402: Conn_01x06, Connector_JST:JST_XH_S6B-XH-A_1x06_P2.50mm_Horizontal, F.Cu at (216.4, 97.5)
- added J501: Conn_ST_STDC14, Connector_PinHeader_1.27mm:PinHeader_2x07_P1.27mm_Vertical_SMD, F.Cu at (196.5, 107.4)
- added J601: Conn_01x03, Connector_JST:JST_XH_S3B-XH-A_1x03_P2.50mm_Horizontal, F.Cu at (216.4, 113.1)
- added J701: Conn_02x05_Odd_FEMALE, Connector_PinSocket_1.27mm:PinSocket_2x05_P1.27mm_Vertical, F.Cu at (240.5, 82.3)
- added J702: Conn_02x05_Odd_FEMALE, Connector_PinSocket_1.27mm:PinSocket_2x05_P1.27mm_Vertical, F.Cu at (245.6, 82.3)
- added J703: Conn_02x05_Odd_FEMALE, Connector_PinSocket_1.27mm:PinSocket_2x05_P1.27mm_Vertical, F.Cu at (250.7, 82.3)
- added JP201: SolderJumper_2_Open, Jumper:SolderJumper-2_P1.3mm_Open_TrianglePad1.0x1.5mm, F.Cu at (194.5, 63.4)
- added JP202: SolderJumper_2_Open, Jumper:SolderJumper-2_P1.3mm_Open_TrianglePad1.0x1.5mm, F.Cu at (194.5, 66.9)
- added JP203: SolderJumper_2_Open, Jumper:SolderJumper-2_P1.3mm_Open_TrianglePad1.0x1.5mm, F.Cu at (194.5, 70.5)
- added JP204: SolderJumper_2_Open, Jumper:SolderJumper-2_P1.3mm_Open_TrianglePad1.0x1.5mm, F.Cu at (194.5, 74.0)
- added L201: 4.7uH, Inductor_SMD:L_0603_1608Metric_Pad1.05x0.95mm_HandSolder, F.Cu at (216.5, 76.4)
- added L501: 47n, Inductor_SMD:L_0603_1608Metric_Pad1.05x0.95mm_HandSolder, F.Cu at (208.5, 93.8)
- added L502: 39n, Inductor_SMD:L_0603_1608Metric_Pad1.05x0.95mm_HandSolder, F.Cu at (208.5, 96.3)
- added L503: 6u, Inductor_SMD:L_0603_1608Metric_Pad1.05x0.95mm_HandSolder, F.Cu at (208.5, 98.9)
- added LED801: RGB, Tom&Jerry:5988G10313F, F.Cu at (260.4, 40.9)
- added LED802: RGB, Tom&Jerry:5988G10313F, F.Cu at (260.4, 46.7)
- added LED803: RGB, Tom&Jerry:5988G10313F, F.Cu at (260.4, 52.5)
- added LED804: RGB, Tom&Jerry:5988G10313F, F.Cu at (260.4, 58.3)
- added PS201: BU33SD5WG-TR, Tom&Jerry:SOT95P280X125-5N, F.Cu at (207.2, 68.0)
- added Q201: PMOS, Tom&Jerry:SOT95P280X125-5N, F.Cu at (207.2, 72.7)
- added R1001: 0.015, Resistor_SMD:R_0402_1005Metric, F.Cu at (264.8, 106.1)
- added R101: 10k, Resistor_SMD:R_0402_1005Metric, F.Cu at (258.7, 64.2)
- added R102: 10k, Resistor_SMD:R_0402_1005Metric, F.Cu at (258.7, 66.2)
- added R103: 10k, Resistor_SMD:R_0402_1005Metric, F.Cu at (258.7, 68.2)
- added R104: 10k, Resistor_SMD:R_0402_1005Metric, F.Cu at (258.7, 70.2)
- added R1201: 10k, Resistor_SMD:R_0402_1005Metric, F.Cu at (265.5, 81.6)
- added R1202: 10k, Resistor_SMD:R_0402_1005Metric, F.Cu at (265.5, 83.6)
- added R1301: 10k, Resistor_SMD:R_0402_1005Metric, F.Cu at (205.9, 115.9)
- added R1302: 10k, Resistor_SMD:R_0402_1005Metric, F.Cu at (205.9, 117.9)
- added R1401: 10k, Resistor_SMD:R_0402_1005Metric, F.Cu at (191.5, 115.9)
- added R1402: 10k, Resistor_SMD:R_0402_1005Metric, F.Cu at (191.5, 117.9)
- added R1501: 10k, Resistor_SMD:R_0402_1005Metric, F.Cu at (265.5, 112.0)
- added R1502: 10k, Resistor_SMD:R_0402_1005Metric, F.Cu at (265.5, 114.0)
- added R201: 100k, Resistor_SMD:R_0402_1005Metric, F.Cu at (201.7, 54.8)
- added R202: 100k, Resistor_SMD:R_0402_1005Metric, F.Cu at (201.7, 56.7)
- added R203: 3.3k, Resistor_SMD:R_0402_1005Metric, F.Cu at (201.7, 58.7)
- added R204: 20, Resistor_SMD:R_0402_1005Metric, F.Cu at (201.7, 60.7)
- added R205: 16k, Resistor_SMD:R_0402_1005Metric, F.Cu at (201.7, 62.7)
- added R206: 7.68k, Resistor_SMD:R_0402_1005Metric, F.Cu at (201.7, 64.7)
- added R207: 40.2k, Resistor_SMD:R_0402_1005Metric, F.Cu at (204.6, 54.8)
- added R208: 3.3k, Resistor_SMD:R_0402_1005Metric, F.Cu at (204.6, 56.7)
- added R209: 3.3k, Resistor_SMD:R_0402_1005Metric, F.Cu at (204.6, 58.7)
- added R210: 3.3k, Resistor_SMD:R_0402_1005Metric, F.Cu at (204.6, 60.7)
- added R211: 3.6k, Resistor_SMD:R_0402_1005Metric, F.Cu at (204.6, 62.7)
- added R212: 27k, Resistor_SMD:R_0402_1005Metric, F.Cu at (204.6, 64.7)
- added R213: 27k, Resistor_SMD:R_0402_1005Metric, F.Cu at (207.5, 54.8)
- added R214: 10k, Resistor_SMD:R_0402_1005Metric, F.Cu at (207.5, 56.7)
- added R215: 15k, Resistor_SMD:R_0402_1005Metric, F.Cu at (207.5, 58.7)
- added R216: 100m, Resistor_SMD:R_0402_1005Metric, F.Cu at (207.5, 60.7)
- added R217: R_Small, Resistor_SMD:R_0402_1005Metric, F.Cu at (207.5, 62.7)
- added R401: 100k, Resistor_SMD:R_0402_1005Metric, F.Cu at (233.9, 81.6)
- added R402: 100k, Resistor_SMD:R_0402_1005Metric, F.Cu at (233.9, 83.6)
- added R501: 100k, Resistor_SMD:R_0402_1005Metric, F.Cu at (203.8, 81.6)
- added R502: 10R, Resistor_SMD:R_0402_1005Metric, F.Cu at (203.8, 83.6)
- added R503: 10k, Resistor_SMD:R_0402_1005Metric, F.Cu at (203.8, 85.6)
- added R504: 10k, Resistor_SMD:R_0402_1005Metric, F.Cu at (203.8, 87.6)
- added R505: 10k, Resistor_SMD:R_0402_1005Metric, F.Cu at (203.8, 89.6)
- added R506: 10k, Resistor_SMD:R_0402_1005Metric, F.Cu at (203.8, 91.6)
- added R901: 0.015, Resistor_SMD:R_0402_1005Metric, F.Cu at (247.4, 124.0)
- added SW501: SW_Push, Button_Switch_SMD:SW_Push_1P1T_NO_6x6mm_H9.5mm, F.Cu at (186.2, 84.4)
- added SW502: SW_Push, Button_Switch_SMD:SW_Push_1P1T_NO_6x6mm_H9.5mm, F.Cu at (186.2, 92.0)
- added SW503: SW_Push, Button_Switch_SMD:SW_Push_1P1T_NO_6x6mm_H9.5mm, F.Cu at (186.2, 99.6)
- added TP201: TestPoint_Small, Test_Point:TestPoint_Pad_D1.5mm, F.Cu at (198.4, 63.4)
- added TP202: TestPoint_Small, Test_Point:TestPoint_Pad_D1.5mm, F.Cu at (198.4, 66.9)
- added TP203: TestPoint_Small, Test_Point:TestPoint_Pad_D1.5mm, F.Cu at (198.4, 70.5)
- added TP204: TestPoint_Small, Test_Point:TestPoint_Pad_D1.5mm, F.Cu at (198.4, 74.0)
- added TP501: PC6, Test_Point:TestPoint_Pad_D1.5mm, F.Cu at (193.4, 82.4)
- added TP502: PB0, Test_Point:TestPoint_Pad_D1.5mm, F.Cu at (193.4, 86.0)
- added TP503: PB1, Test_Point:TestPoint_Pad_D1.5mm, F.Cu at (193.4, 89.5)
- added TP504: PB4, Test_Point:TestPoint_Pad_D1.5mm, F.Cu at (193.4, 93.1)
- added TP505: PB5, Test_Point:TestPoint_Pad_D1.5mm, F.Cu at (193.4, 96.6)
- added TP506: PB6, Test_Point:TestPoint_Pad_D1.5mm, F.Cu at (193.4, 100.2)
- added TP507: PB10, Test_Point:TestPoint_Pad_D1.5mm, F.Cu at (197.0, 82.4)
- added TP508: PB11, Test_Point:TestPoint_Pad_D1.5mm, F.Cu at (197.0, 86.0)
- added TP509: PA0, Test_Point:TestPoint_Pad_D1.5mm, F.Cu at (197.0, 89.5)
- added TP510: PA1, Test_Point:TestPoint_Pad_D1.5mm, F.Cu at (197.0, 93.1)
- added TP511: PA4, Test_Point:TestPoint_Pad_D1.5mm, F.Cu at (197.0, 96.6)
- added TP512: PA6, Test_Point:TestPoint_Pad_D1.5mm, F.Cu at (197.0, 100.2)
- added TP513: PA7, Test_Point:TestPoint_Pad_D1.5mm, F.Cu at (200.6, 82.4)
- added TP514: PA9, Test_Point:TestPoint_Pad_D1.5mm, F.Cu at (200.6, 86.0)
- added TP515: PA10, Test_Point:TestPoint_Pad_D1.5mm, F.Cu at (200.6, 89.5)
- added TP516: PA11, Test_Point:TestPoint_Pad_D1.5mm, F.Cu at (200.6, 93.1)
- added TP517: PA12, Test_Point:TestPoint_Pad_D1.5mm, F.Cu at (200.6, 96.6)
- added U1001: ZXBM5210-S, Tom&Jerry:XBM5210, F.Cu at (263.6, 101.8)
- added U201: MP1475DJ-LF-P, Tom&Jerry:SOT65P280X100-8N, F.Cu at (217.5, 67.9)
- added U202: BQ25172DSGR, Tom&Jerry:IC_BQ25172DSGR, F.Cu at (207.1, 76.8)
- added U301: ADXL343, Tom&Jerry:PQFN80P300X500X100-14N, F.Cu at (233.5, 61.6)
- added U501: STM32G431CBU6, Package_DFN_QFN:QFN-48-1EP_7x7mm_P0.5mm_EP5.1x5.1mm, F.Cu at (205.9, 106.6)
- added U601: PAM8302AAY, Tom&Jerry:DFN300X300X80-8N, F.Cu at (216.3, 125.6)
- added U801: LP5812ADSDR, Tom&Jerry:WSON8_DSD_TEX, F.Cu at (266.7, 40.4)
- added U901: ZXBM5210-S, Tom&Jerry:XBM5210, F.Cu at (246.2, 119.8)
- added Y501: 16MHz, Crystal:Crystal_SMD_3225-4Pin_3.2x2.5mm, F.Cu at (183.2, 105.6)
- moved H1102 29.7 mm to (124.0, 110.4)
- moved H1104 29.7 mm to (78.0, 110.4)
- moved H1101 29.7 mm to (124.0, 61.4)
- moved H1103 29.7 mm to (78.0, 61.4)
- renumbered H1601 to H1101, H1602 to H1102, H1603 to H1103, H1604 to H1104

Commit message: First try placement
Parts:
- removed TP201, TP202, TP203, TP204: TestPoint_Small, Test_Point:TestPoint_Pad_D1.5mm
- moved R1001 185.8 mm to (80.5, 81.8), turned to -90 degrees
- moved U1001 183.1 mm to (82.5, 74.8), turned to 90 degrees
- moved C1003 179.9 mm to (80.3, 69.1), turned to 90 degrees
- moved C1005 179.3 mm to (87.5, 80.8), turned to -90 degrees
- moved IC1001 177.8 mm to (85.0, 81.3), turned to 180 degrees
- moved C1002 177.0 mm to (80.5, 84.5), turned to -90 degrees
- moved C1001 176.8 mm to (82.5, 69.1), turned to 90 degrees
- moved C1004 175.6 mm to (82.5, 84.5), turned to -90 degrees
- moved R901 168.6 mm to (80.5, 100.3), turned to -90 degrees
- moved U901 165.9 mm to (82.5, 93.3), turned to 90 degrees
- moved C903 162.7 mm to (80.5, 87.8), turned to 90 degrees
- moved C905 161.6 mm to (88.0, 99.5), turned to -90 degrees
- moved IC901 160.1 mm to (85.5, 99.9), turned to 180 degrees
- moved C901 159.7 mm to (82.5, 87.8), turned to 90 degrees
- moved C904 158.9 mm to (82.0, 103.3), turned to -90 degrees
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
Commit message: Try some placement and routing
Parts:
- removed C509: 100n, Capacitor_SMD:C_0402_1005Metric
- removed H1104: MountingHole_Pad, MountingHole:MountingHole_3.2mm_M3_Pad_Via
- removed L503: 6u, Inductor_SMD:L_0603_1608Metric_Pad1.05x0.95mm_HandSolder
- removed TP501: PC6, Test_Point:TestPoint_Pad_D1.5mm
- removed TP502: PB0, Test_Point:TestPoint_Pad_D1.5mm
- removed TP503: PB1, Test_Point:TestPoint_Pad_D1.5mm
- removed TP504: PB4, Test_Point:TestPoint_Pad_D1.5mm
- removed TP505: PB5, Test_Point:TestPoint_Pad_D1.5mm
- removed TP506: PB6, Test_Point:TestPoint_Pad_D1.5mm
- removed TP507: PB10, Test_Point:TestPoint_Pad_D1.5mm
- removed TP508: PB11, Test_Point:TestPoint_Pad_D1.5mm
- removed TP509: PA0, Test_Point:TestPoint_Pad_D1.5mm
- removed TP510: PA1, Test_Point:TestPoint_Pad_D1.5mm
- removed TP511: PA4, Test_Point:TestPoint_Pad_D1.5mm
- removed TP512: PA6, Test_Point:TestPoint_Pad_D1.5mm
- removed TP513: PA7, Test_Point:TestPoint_Pad_D1.5mm
- removed TP514: PA9, Test_Point:TestPoint_Pad_D1.5mm
- removed TP515: PA10, Test_Point:TestPoint_Pad_D1.5mm
- removed TP516: PA11, Test_Point:TestPoint_Pad_D1.5mm
- removed TP517: PA12, Test_Point:TestPoint_Pad_D1.5mm
- moved H1601 205.3 mm to (225.6, 80.0)
- moved H1602 205.3 mm to (225.6, 88.0)
- moved H701 205.3 mm to (215.7, 80.0)
- moved H702 205.3 mm to (215.7, 88.0)
- moved LED801 171.0 mm to (101.7, 104.6), turned to 180 degrees
- moved R103 168.4 mm to (93.0, 98.3), turned to 90 degrees
- moved U801 165.8 mm to (112.0, 100.0)
- moved LED802 163.8 mm to (107.2, 104.6)
- moved R101 162.6 mm to (98.0, 89.0), turned to 180 degrees
- moved R102 162.5 mm to (99.0, 96.0), turned to 180 degrees
- moved R104 161.6 mm to (99.0, 95.0), turned to 180 degrees
- moved LED803 156.9 mm to (112.4, 104.6), turned to 180 degrees
- moved R1201 154.2 mm to (113.5, 107.5)
- moved R1202 151.9 mm to (115.5, 107.5), turned to 180 degrees
- moved LED804 149.8 mm to (117.9, 104.6), turned to 180 degrees
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Routing:
- net Net-(D206-K): track 0.00 -> 45.4 mm
- net /Périphériques/LIDAR_TX: track 0.00 -> 39.3 mm
- net /Périphériques/LIDAR_RX: track 0.00 -> 37.7 mm
- net /Musique/DAC_STM+: track 0.00 -> 37.1 mm, vias 0 -> 2
- net +3.3V: track 0.00 -> 32.5 mm
- net /STM32/NRST: track 0.00 -> 32.4 mm
- net /STM32/STLINK_SWO: track 0.00 -> 25.4 mm, vias 0 -> 2
- net Net-(JP201-A): track 0.00 -> 23.0 mm
- net +5V: track 0.00 -> 22.2 mm
- net /STM32/VCP_TX: track 0.00 -> 22.2 mm, vias 0 -> 2
- net /STM32/STLINK_SWDIO: track 0.00 -> 19.9 mm
- net /STM32/STLINK_SWCLK: track 0.00 -> 19.7 mm
- net Net-(D205-K): track 0.00 -> 19.1 mm
- net /Alimentation/Batt_CHG: track 0.00 -> 18.5 mm
- net +3.3VA: track 0.00 -> 17.8 mm
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