File: electronique/schematic_draft/tom&Jerry_Draft/Charger.kicad_sch (KiCad schematic)
At the start: 54 parts, among them J201 Interrupteur, Q201 PMOS

Commit message: Ajout des bonnes empreintes
Parts:
- Q201: footprint (none) -> Tom&Jerry:SOT95P280X125-5N
Changed lines of the file:
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@@
 			)
 		)
-		(property "Footprint" ""
+		(property "Footprint" "Tom&Jerry:SOT95P280X125-5N"
 			(at 262.89 82.55 0)
 			(effects

Commit message: Ajout V2 TOF + MultiPCB Panalize
Parts:
- renumbered C212 to C203, C213 to C208, C206 to C210, C207 to C211, C211 to C212, D205 to D201, D204 to D202, D206 to D203, D207 to D204, J201 to J204, R215 to R203, R214 to R208, R216 to R209, R217 to R210, R210 to R211, R211 to R212, R212 to R213, R213 to R214, R208 to R215, R202 to R216, R209 to R217, TP202 to TP201, TP201 to TP202

Commit message: V2.0 placement avec tout dessus
Aucun routage réalisé
Parts:
- removed TP201, TP202, TP203, TP204: TestPoint_Small, Test_Point:TestPoint_Pad_D1.5mm, symbol Connector:TestPoint_Small

Commit message: Routage Signal Complet - PCB V2.0
Parts:
- renumbered C210 to C206, C211 to C207, C212 to C211, C203 to C212, C208 to C213, D202 to D204, D201 to D205, D203 to D206, D204 to D207, J204 to J201, R216 to R202, R215 to R208, R217 to R209, R211 to R210, R212 to R211, R213 to R212, R214 to R213, R208 to R214, R203 to R215, R209 to R216, R210 to R217
