File: electronique/schematic_draft/tom&Jerry_Draft/Charger.kicad_sch (KiCad schematic)
At the start: 50 parts, among them J201 Interrupteur, Q201 SI2365EDS-T1-GE3

Commit message: Nothing important, just an inchident
Parts:
- Q201: footprint SOT95P237X112-3N -> Tom&Jerry:SOT95P237X112-3N
Changed lines of the file:
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@@
 			)
 		)
-		(property "Footprint" "SOT95P237X112-3N"
+		(property "Footprint" "Tom&Jerry:SOT95P237X112-3N"
 			(at 264.16 -18.72 0)
 			(effects
