File: electronique/schematic_draft/tom&Jerry_Draft/Moustache.kicad_sch (KiCad schematic)
At the start: 8 parts, among them IC301 TCA9555RTWR, J301 FTSH-105-01-F-DV-P-TR, J302 FTSH-105-01-F-DV-P-TR, J303 FTSH-105-01-F-DV-P-TR, J304 FTSH-105-01-F-DV-P-TR, J305 Conn_01x08, U301 ADXL343

Commit message: Routage Signal Complet
Connections:
- net LIDAR_DEV_EN: now also IC301.14 (P14); no longer IC301.15 (P15)
- net LIDAR_M_EN: now also IC301.15 (P15); no longer IC301.14 (P14)
- net TOF1_GPIO1: now also IC301.8 (P07); no longer IC301.7 (P06)
- net TOF1_XSHUT: now also IC301.7 (P06); no longer IC301.8 (P07)
- net TOF4_XSHUT: now also IC301.3 (P02); no longer IC301.1 (P00)
- net TOF5_XSHUT: now also IC301.1 (P00); no longer IC301.3 (P02)
Changed lines of the file:
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@@
 		)
 	)
-	(label "TOF1_XSHUT"
+	(label "TOF1_GPIO1"
 		(at 44.45 152.4 180)
 		(fields_autoplaced yes)
@@
 		)
 	)
-	(label "TOF1_GPIO1"
+	(label "TOF1_XSHUT"
 		(at 44.45 149.86 180)
 		(fields_autoplaced yes)
@@
 		)
 	)
-	(label "LIDAR_M_EN"
+	(label "LIDAR_DEV_EN"
 		(at 66.04 173.99 270)
 		(fields_autoplaced yes)
@@
 		)
 	)
-	(label "TOF5_XSHUT"
+	(label "TOF4_XSHUT"
 		(at 71.12 138.43 90)
 		(fields_autoplaced yes)
@@
 		)
 	)
-	(label "LIDAR_DEV_EN"
+	(label "LIDAR_M_EN"
 		(at 68.58 173.99 270)
 		(fields_autoplaced yes)
@@
 		)
 	)
-	(label "TOF4_XSHUT"
+	(label "TOF5_XSHUT"
 		(at 76.2 138.43 90)
 		(fields_autoplaced yes)

Commit message: Routage Signal Complet - PCB V2.0
Parts:
- removed J301, J302, J303, J304: FTSH-105-01-F-DV-P-TR, Tom&Jerry:SAMTEC_FTSH-105-01-F-DV-P-TR, symbol Tom&Jerry:FTSH-105-01-F-DV-P-TR
- renumbered J305 to J301
Connections:
- net IMU_INT1: now also IC301.16 (P16); no longer IC301.17 (P17)
- net IMU_INT2: now also IC301.17 (P17); no longer IC301.16 (P16)
- net LIDAR_DEV_EN: now also IC301.15 (P15); no longer IC301.14 (P14)
- net LIDAR_M_EN: now also IC301.14 (P14); no longer IC301.15 (P15)
- net TOF4_GPIO1: now also IC301.5 (P04); no longer IC301.2 (P01)
- net TOF4_XSHUT: now also IC301.6 (P05); no longer IC301.3 (P02)
- net TOF5_GPIO1: now also IC301.3 (P02); no longer IC301.4 (P03)
- net TOF5_XSHUT: now also IC301.4 (P03); no longer IC301.1 (P00)
- net TOF6_GPIO1: now also IC301.2 (P01); no longer IC301.6 (P05)
- net TOF6_XSHUT: now also IC301.1 (P00); no longer IC301.5 (P04)
Other:
- removed sheet TOF7
- removed sheet TOF8
- added sheet TOF NORD (TOF_PCB.kicad_sch)
- added sheet TOF SUD (TOF_PCB.kicad_sch)
