File: electronique/Tom&Jerry_PCB/Charger.kicad_sch (KiCad schematic)
At the start: 50 parts, among them J201 Interrupteur, Q201 SI2365EDS-T1-GE3

Commit message: Adding all files to critic error PCB
Parts:
- R209: value R_Small -> 3.3k
Other:
- removed sheet Battery Charging LEDs

Commit message: MAJOR UPGRADE : cubeIDE rtos - multiple drivers work | MINOR UPGRADE : schematic correction (too late)| COMMIT BEFORE MULTIPLE TASKS CREATION
Parts:
- R202: value 100m -> 110m
- R210: value 3.6k -> 3.3k
- R214: value 3.3k -> 300
Changed lines of the file:
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@@
 			)
 		)
-		(property "Value" "3.3k"
+		(property "Value" "300"
 			(at 116.84 172.72 90)
 			(effects
@@
 			)
 		)
-		(property "Value" "3.6k"
+		(property "Value" "3.3k"
 			(at 176.53 134.6199 0)
 			(effects
@@
 			)
 		)
-		(property "Value" "100m"
+		(property "Value" "110m"
 			(at 251.46 59.6899 0)
 			(effects
