File: electronique/Tom&Jerry_PCB/musique.kicad_sch (KiCad schematic)
At the start: 11 parts, among them J601 Conn_01x03, U601 PAM8302AAY

Commit message: MAJOR UPGRADE : cubeIDE rtos - multiple drivers work | MINOR UPGRADE : schematic correction (too late)| COMMIT BEFORE MULTIPLE TASKS CREATION
Parts:
- U601: now not fitted
Changed lines of the file:
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@@
 		(in_bom yes)
 		(on_board yes)
-		(dnp no)
+		(dnp yes)
 		(property "Reference" "U601"
 			(at 136.8141 78.74 0)
