File: electronique/Tom&Jerry_PCB/Moustache.kicad_sch (KiCad schematic)
At the start: 4 parts, among them IC301 TCA9555RTWR, J301 Conn_01x08, U301 ADXL343

Commit message: Adding all files to critic error PCB
Parts:
- added C302: 0.1u, Capacitor_SMD:C_0603_1608Metric, symbol Device:C_Small
- C301: footprint Capacitor_SMD:C_0805_2012Metric -> Capacitor_SMD:C_0402_1005Metric
Connections:
- net +3.3V: now also C302.1
- net GND: now also C302.2
Other:
- moved on the sheet: C301

Commit message: MAJOR UPGRADE : cubeIDE rtos - multiple drivers work | MINOR UPGRADE : schematic correction (too late)| COMMIT BEFORE MULTIPLE TASKS CREATION
Parts:
- C302: value 0.1u -> 100n
Changed lines of the file:
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@@
 			)
 		)
-		(property "Value" "0.1u"
+		(property "Value" "100n"
 			(at 233.68 36.8362 0)
 			(effects

Commit message: Ajout bonne bobines + 3.3v gpio expander + Driver moteur
Connections:
- net +3.3V: now also IC301.21 (VCC)
- net +5V: no longer IC301.21 (VCC)
Changed lines of the file:
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@@
 	(wire
 		(pts
-			(xy 93.98 158.75) (xy 90.17 158.75)
+			(xy 90.17 158.75) (xy 101.6 158.75)
 		)
 		(stroke
@@
 	)
 	(symbol
+		(lib_name "+3.3V_1")
+		(lib_id "power:+3.3V")
+		(at 101.6 158.75 270)
+		(unit 1)
+		(exclude_from_sim no)
+		(in_bom yes)
+		(on_board yes)
+		(dnp no)
+		(fields_autoplaced yes)
+		(property "Reference" "#PWR0312"
+			(at 97.79 158.75 0)
+			(effects
+				(font
+					(size 1.27 1.27)
+				)
+				(hide yes)
+			)
+		)
+		(property "Value" "+3.3V"
+			(at 105.41 158.7499 90)
+			(effects
+				(font
+					(size 1.27 1.27)
+				)
+				(justify left)
+			)
+		)
+		(property "Footprint" ""
+			(at 101.6 158.75 0)
+			(effects
+				(font
+					(size 1.27 1.27)
+				)
+				(hide yes)
+			)
+		)
+		(property "Datasheet" ""
+			(at 101.6 158.75 0)
+			(effects
+				(font
+					(size 1.27 1.27)
+				)
+				(hide yes)
+			)
+		)
+		(property "Description" "Power symbol creates a global label with name \"+3.3V\""
+			(at 101.6 158.75 0)
+			(effects
+				(font
+					(size 1.27 1.27)
+				)
+				(hide yes)
+			)
+		)
+		(pin "1"
+		)
+		(instances
+			(project "Tom&Jerry_PCB"
+				(path "/d6e3fbeb-d028-494d-83bf-2e4a8b12578d/ac7f7f04-c418-4551-b204-a999b9c3c440"
+					(reference "#PWR0312")
+					(unit 1)
+				)
+			)
+		)
+	)
+	(symbol
 		(lib_name "GND_3")
 		(lib_id "power:GND")
@@
 					(unit 1)
 				)
-			)
-		)
-	)
-	(symbol
-		(lib_id "power:+5V")
-		(at 93.98 158.75 0)
-		(unit 1)
-		(exclude_from_sim no)
-		(in_bom yes)
-		(on_board yes)
-		(dnp no)
-		(fields_autoplaced yes)
-		(property "Reference" "#PWR0310"
-			(at 93.98 162.56 0)
-			(effects
-				(font
-					(size 1.27 1.27)
-				)
-				(hide yes)
-			)
-		)
-		(property "Value" "+5V"
-			(at 96.52 157.4799 0)
-			(effects
-				(font
-					(size 1.27 1.27)
-				)
-				(justify left)
-			)
-		)
-		(property "Footprint" ""
-			(at 93.98 158.75 0)
-			(effects
-				(font
-					(size 1.27 1.27)
-				)
-				(hide yes)
-			)
-		)
-		(property "Datasheet" ""
-			(at 93.98 158.75 0)
-			(effects
-				(font
-					(size 1.27 1.27)
-				)
-				(hide yes)
-			)
-		)
-		(property "Description" "Power symbol creates a global label with name \"+5V\""
-			(at 93.98 158.75 0)
-			(effects
-				(font
-					(size 1.27 1.27)
-				)
-				(hide yes)
-			)
-		)
-		(pin "1"
-		)
-		(instances
-			(project "Tom&Jerry_PCB"
-				(path "/d6e3fbeb-d028-494d-83bf-2e4a8b12578d/ac7f7f04-c418-4551-b204-a999b9c3c440"
-					(reference "#PWR0310")
-					(unit 1)
-				)
