File: electronique/Tom&Jerry_PCB/STM32x.kicad_sch (KiCad schematic)
At the start: 26 parts, among them J501 Conn_ST_STDC14, SW501 SW_Push, SW502 SW_Push, SW503 SW_Push, U501 STM32G431CBU6, Y501 16MHz

Commit message: Ajout bonne bobines + 3.3v gpio expander + Driver moteur
Parts:
- L501: footprint Inductor_SMD:L_0603_1608Metric_Pad1.05x0.95mm_HandSolder -> Tom&Jerry:WE-LQS_2512
Changed lines of the file:
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@@
 			)
 		)
-		(property "Footprint" "Inductor_SMD:L_0603_1608Metric_Pad1.05x0.95mm_HandSolder"
+		(property "Footprint" "Tom&Jerry:WE-LQS_2512"
 			(at 73.66 44.45 0)
 			(effects
