File: electronique/Tom&Jerry_PCB/Tom&Jerry_PCB.kicad_pcb (KiCad board)
At the start: 4 copper layers, 54 x 57 mm, 146 parts, among them IC1101 NCS199A2RSQT2G, IC301 TCA9555RTWR, IC901 NCS199A2RSQT2G, J1001 FTSH-105-01-F-DV-P-TR, J1301 Conn_01x02, J1501 Conn_01x02, J1601 Conn_01x02, J1701 Conn_01x02, J201 Interrupteur, J202 USB_C_Receptacle_USB2.0_16P, J203 Conn_01x02, J204 Conn_01x02, J301 Conn_01x08, J401 Conn_01x06, J402 Conn_01x06, J501 Conn_ST_STDC14, J601 Conn_01x03, J701 FTSH-105-01-F-DV-P-TR, Q201 SI2365EDS-T1-GE3, SW501 SW_Push, SW502 SW_Push, SW503 SW_Push, U1101 ZXBM5210-S, U201 MP1475DJ-LF-P, U202 BQ25172DSGR, U301 ADXL343, U501 STM32G431CBU6, U601 PAM8302AAY, U801 LP5812ADSDR, U901 ZXBM5210-S, Y501 16MHz

Commit message: Ajout bonne bobines + 3.3v gpio expander + Driver moteur
Parts:
- C302: value 0.1u -> 100n
- L501: footprint Inductor_SMD:L_0603_1608Metric_Pad1.05x0.95mm_HandSolder -> Tom&Jerry:WE-LQS_2512
- R202: value 100m -> 110m
- R210: value 3.6k -> 3.3k
- R214: value 3.3k -> 300
- moved L501 4.42 mm to (96.0, 90.2)
Connections:
- IC301 pad 21: +5V -> +3.3V
- IC301 pad 25: GND -> (no net)
- IC301 pad V: GND -> (no net)
- U1101 pad 9: GND -> (no net)
- U202 pad 10: GND -> (no net)
- U202 pad 11: GND -> (no net)
- U601 pad 9: GND -> (no net)
- U901 pad 9: GND -> (no net)
Routing:
- net +3.3V: track 114.3 -> 141.4 mm, vias 27 -> 34
- net +5V: track 117.8 -> 119.1 mm
- net GND: vias 101 -> 100
